Commit message: init

File: output/label13.urdf (robot description, URDF)
Before this commit: robot my_urdf, 9 links, 8 joints
Links:
- removed link doorL2
- removed link doorR3
- removed link drawer0
- removed link drawer1
- added link doorL1, mass 0.2; collision mesh filename=../meshes/parts/doorL.obj scale=1 1.99 2.99; visual mesh filename=../meshes/parts/doorL.obj scale=1 1.99 2.99
- added link doorR0, mass 0.2; collision mesh filename=../meshes/parts/doorR.obj scale=1 1.99 2.99; visual mesh filename=../meshes/parts/doorR.obj scale=1 1.99 2.99
- added link drawer2, mass 0.2; collision mesh filename=../meshes/parts/drawer.obj scale=1 1.98 0.98; visual mesh filename=../meshes/parts/drawer.obj scale=1 1.98 0.98
- added link drawer3, mass 0.2; collision mesh filename=../meshes/parts/drawer.obj scale=1 1.98 0.98; visual mesh filename=../meshes/parts/drawer.obj scale=1 1.98 0.98
Joints:
- removed joint doorL2_to_base_link
- removed joint doorR3_to_base_link
- removed joint drawer0_to_base_link
- removed joint drawer1_to_base_link
- removed joint handle4_to_drawer0
- removed joint handle5_to_drawer1
- removed joint knob6_to_doorL2
- removed joint knob7_to_doorR3
- added joint doorL1_to_base_link: type revolute, parent base_link, child doorL1, origin xyz=0 0.0 0.0 rpy=0.0 0.0 0.0, axis 0 0 1, limit lower=-1.57 upper=0 effort=5 velocity=2.283
- added joint doorR0_to_base_link: type revolute, parent base_link, child doorR0, origin xyz=0 1.0 0.0 rpy=-0.0 -0.0 -0.0, axis 0 0 1, limit lower=0 upper=1.57 effort=5 velocity=2.283
- added joint drawer2_to_base_link: type prismatic, parent base_link, child drawer2, origin xyz=0 0.0 0.75 rpy=0.0 0.0 0.0, axis 1 0 0, limit lower=0 upper=0.4 effort=5 velocity=2.283
- added joint drawer3_to_base_link: type prismatic, parent base_link, child drawer3, origin xyz=0 0.5 0.75 rpy=0.0 0.0 0.0, axis 1 0 0, limit lower=0 upper=0.4 effort=5 velocity=2.283
- added joint handle4_to_drawer3: type fixed, parent drawer3, child handle4, origin xyz=0 0.25 0.125 rpy=1.5707963267948963 0.0 0.0, axis 0 0 1, limit lower=0 upper=1.57 effort=5 velocity=2.283
- added joint handle5_to_drawer2: type fixed, parent drawer2, child handle5, origin xyz=0 0.25 0.125 rpy=1.5707963267948963 0.0 0.0, axis 0 0 1, limit lower=0 upper=1.57 effort=5 velocity=2.283
- added joint knob6_to_doorL1: type fixed, parent doorL1, child knob6, origin xyz=0 0.4166666666666667 0.375 rpy=0.0 0.0 0.0, axis 1 0 0, limit lower=0 upper=1.57 effort=5 velocity=2.283
- added joint knob7_to_doorR0: type fixed, parent doorR0, child knob7, origin xyz=0 -0.4166666666666667 0.375 rpy=0.0 0.0 0.0, axis 1 0 0, limit lower=0 upper=1.57 effort=5 velocity=2.283

File: output/label29.urdf (robot description, URDF)
Before this commit: robot my_urdf, 9 links, 8 joints
Links:
- removed link doorL3
- removed link doorR2
- removed link drawer0
- removed link drawer1
- added link doorL0, mass 0.2; collision mesh filename=../meshes/parts/doorL.obj scale=1 1.99 2.99; visual mesh filename=../meshes/parts/doorL.obj scale=1 1.99 2.99
- added link doorR1, mass 0.2; collision mesh filename=../meshes/parts/doorR.obj scale=1 1.99 2.99; visual mesh filename=../meshes/parts/doorR.obj scale=1 1.99 2.99
- added link drawer2, mass 0.2; collision mesh filename=../meshes/parts/drawer.obj scale=1 1.98 0.98; visual mesh filename=../meshes/parts/drawer.obj scale=1 1.98 0.98
- added link drawer3, mass 0.2; collision mesh filename=../meshes/parts/drawer.obj scale=1 1.98 0.98; visual mesh filename=../meshes/parts/drawer.obj scale=1 1.98 0.98
Joints:
- removed joint doorL3_to_base_link
- removed joint doorR2_to_base_link
- removed joint drawer0_to_base_link
- removed joint drawer1_to_base_link
- removed joint knob4_to_drawer0
- removed joint knob5_to_drawer1
- removed joint knob6_to_doorR2
- removed joint knob7_to_doorL3
- added joint doorL0_to_base_link: type revolute, parent base_link, child doorL0, origin xyz=0 0.0 0.0 rpy=0.0 0.0 0.0, axis 0 0 1, limit lower=-1.57 upper=0 effort=5 velocity=2.283
- added joint doorR1_to_base_link: type revolute, parent base_link, child doorR1, origin xyz=0 1.0 0.0 rpy=-0.0 -0.0 -0.0, axis 0 0 1, limit lower=0 upper=1.57 effort=5 velocity=2.283
- added joint drawer2_to_base_link: type prismatic, parent base_link, child drawer2, origin xyz=0 0.5 0.75 rpy=0.0 0.0 0.0, axis 1 0 0, limit lower=0 upper=0.4 effort=5 velocity=2.283
- added joint drawer3_to_base_link: type prismatic, parent base_link, child drawer3, origin xyz=0 0.0 0.75 rpy=0.0 0.0 0.0, axis 1 0 0, limit lower=0 upper=0.4 effort=5 velocity=2.283
- added joint knob4_to_drawer3: type fixed, parent drawer3, child knob4, origin xyz=0 0.25 0.125 rpy=1.5707963267948963 0.0 0.0, axis 0 0 1, limit lower=0 upper=1.57 effort=5 velocity=2.283
- added joint knob5_to_drawer2: type fixed, parent drawer2, child knob5, origin xyz=0 0.25 0.125 rpy=1.5707963267948963 0.0 0.0, axis 0 0 1, limit lower=0 upper=1.57 effort=5 velocity=2.283
- added joint knob6_to_doorR1: type fixed, parent doorR1, child knob6, origin xyz=0 -0.4166666666666667 0.375 rpy=0.0 0.0 0.0, axis 1 0 0, limit lower=0 upper=1.57 effort=5 velocity=2.283
- added joint knob7_to_doorL0: type fixed, parent doorL0, child knob7, origin xyz=0 0.4166666666666667 0.375 rpy=0.0 0.0 0.0, axis 1 0 0, limit lower=0 upper=1.57 effort=5 velocity=2.283

File: output/label3.urdf (robot description, URDF)
Before this commit: robot my_urdf, 11 links, 10 joints
Links:
- link drawer1: geometry collision mesh filename=../meshes/parts/drawer.obj scale=1 1.98 0.6466666666666666; visual mesh filename=../meshes/parts/drawer.obj scale=1 1.98 0.6466666666666666
- link drawer2: geometry collision mesh filename=../meshes/parts/drawer.obj scale=1 1.98 0.98; visual mesh filename=../meshes/parts/drawer.obj scale=1 1.98 0.98
Joints:
- removed joint knob5_to_drawer0
- removed joint knob6_to_drawer1
- removed joint knob7_to_drawer2
- added joint knob5_to_drawer2: type fixed, parent drawer2, child knob5, origin xyz=0 0.25 0.125 rpy=1.5707963267948963 0.0 0.0, axis 0 0 1, limit lower=0 upper=1.57 effort=5 velocity=2.283
- added joint knob6_to_drawer0: type fixed, parent drawer0, child knob6, origin xyz=0 0.25 0.125 rpy=1.5707963267948963 0.0 0.0, axis 0 0 1, limit lower=0 upper=1.57 effort=5 velocity=2.283
- added joint knob7_to_drawer1: type fixed, parent drawer1, child knob7, origin xyz=0 0.25 0.08333333333333333 rpy=1.5707963267948963 0.0 0.0, axis 0 0 1, limit lower=0 upper=1.57 effort=5 velocity=2.283
- joint drawer0_to_base_link: origin xyz=0 0.0 0.75 rpy=0.0 0.0 0.0 -> xyz=0 0.0 0.5 rpy=0.0 0.0 0.0
- joint drawer1_to_base_link: origin xyz=0 0.0 0.5 rpy=0.0 0.0 0.0 -> xyz=0 0.0 0.3333333333333333 rpy=0.0 0.0 0.0
- joint drawer2_to_base_link: origin xyz=0 0.0 0.3333333333333333 rpy=0.0 0.0 0.0 -> xyz=0 0.0 0.75 rpy=0.0 0.0 0.0

File: output/label4.urdf (robot description, URDF)
Before this commit: robot my_urdf, 5 links, 4 joints
Joints:
- removed joint knob2_to_doorR0
- removed joint knob3_to_doorR1
- added joint knob2_to_doorR1: type fixed, parent doorR1, child knob2, origin xyz=0 -0.8333333333333334 0.25 rpy=0.0 0.0 0.0, axis 1 0 0, limit lower=0 upper=1.57 effort=5 velocity=2.283
- added joint knob3_to_doorR0: type fixed, parent doorR0, child knob3, origin xyz=0 -0.8333333333333334 0.25 rpy=0.0 0.0 0.0, axis 1 0 0, limit lower=0 upper=1.57 effort=5 velocity=2.283
- joint doorR0_to_base_link: origin xyz=0 1.0 0.0 rpy=-0.0 -0.0 -0.0 -> xyz=0 1.0 0.5 rpy=-0.0 -0.0 -0.0
- joint doorR1_to_base_link: origin xyz=0 1.0 0.5 rpy=-0.0 -0.0 -0.0 -> xyz=0 1.0 0.0 rpy=-0.0 -0.0 -0.0

File: output/label40.urdf (robot description, URDF)
Before this commit: robot my_urdf, 17 links, 16 joints
Links:
- removed link doorL6
- removed link doorR7
- removed link drawer0
- removed link drawer1
- added link doorL1, mass 0.2; collision mesh filename=../meshes/parts/doorL.obj scale=1 1.3233333333333333 2.99; visual mesh filename=../meshes/parts/doorL.obj scale=1 1.3233333333333333 2.99
- added link doorR0, mass 0.2; collision mesh filename=../meshes/parts/doorR.obj scale=1 1.3233333333333333 2.99; visual mesh filename=../meshes/parts/doorR.obj scale=1 1.3233333333333333 2.99
- added link drawer6, mass 0.2; collision mesh filename=../meshes/parts/drawer.obj scale=1 1.3133333333333332 0.98; visual mesh filename=../meshes/parts/drawer.obj scale=1 1.3133333333333332 0.98
- added link drawer7, mass 0.2; collision mesh filename=../meshes/parts/drawer.obj scale=1 1.3133333333333332 0.98; visual mesh filename=../meshes/parts/drawer.obj scale=1 1.3133333333333332 0.98
Joints:
- removed joint doorL6_to_base_link
- removed joint doorR7_to_base_link
- removed joint drawer0_to_base_link
- removed joint drawer1_to_base_link
- removed joint handle10_to_drawer2
- removed joint handle11_to_drawer3
- removed joint handle12_to_drawer4
- removed joint handle13_to_drawer5
- removed joint handle14_to_doorL6
- removed joint handle15_to_doorR7
- removed joint handle8_to_drawer0
- removed joint handle9_to_drawer1
- added joint doorL1_to_base_link: type revolute, parent base_link, child doorL1, origin xyz=0 0.0 0.0 rpy=0.0 0.0 0.0, axis 0 0 1, limit lower=-1.57 upper=0 effort=5 velocity=2.283
- added joint doorR0_to_base_link: type revolute, parent base_link, child doorR0, origin xyz=0 1.0 0.0 rpy=-0.0 -0.0 -0.0, axis 0 0 1, limit lower=0 upper=1.57 effort=5 velocity=2.283
- added joint drawer6_to_base_link: type prismatic, parent base_link, child drawer6, origin xyz=0 0.6666666666666666 0.75 rpy=0.0 0.0 0.0, axis 1 0 0, limit lower=0 upper=0.4 effort=5 velocity=2.283
- added joint drawer7_to_base_link: type prismatic, parent base_link, child drawer7, origin xyz=0 0.0 0.75 rpy=0.0 0.0 0.0, axis 1 0 0, limit lower=0 upper=0.4 effort=5 velocity=2.283
- added joint handle10_to_drawer5: type fixed, parent drawer5, child handle10, origin xyz=0 0.16666666666666666 0.125 rpy=1.5707963267948963 0.0 0.0, axis 0 0 1, limit lower=0 upper=1.57 effort=5 velocity=2.283
- added joint handle11_to_drawer4: type fixed, parent drawer4, child handle11, origin xyz=0 0.16666666666666666 0.125 rpy=1.5707963267948963 0.0 0.0, axis 0 0 1, limit lower=0 upper=1.57 effort=5 velocity=2.283
- added joint handle12_to_drawer3: type fixed, parent drawer3, child handle12, origin xyz=0 0.16666666666666666 0.125 rpy=1.5707963267948963 0.0 0.0, axis 0 0 1, limit lower=0 upper=1.57 effort=5 velocity=2.283
- added joint handle13_to_drawer2: type fixed, parent drawer2, child handle13, origin xyz=0 0.16666666666666666 0.125 rpy=1.5707963267948963 0.0 0.0, axis 0 0 1, limit lower=0 upper=1.57 effort=5 velocity=2.283
- added joint handle14_to_doorL1: type fixed, parent doorL1, child handle14, origin xyz=0 0.2777777777777778 0.375 rpy=0.0 0.0 0.0, axis 1 0 0, limit lower=0 upper=1.57 effort=5 velocity=2.283
- added joint handle15_to_doorR0: type fixed, parent doorR0, child handle15, origin xyz=0 -0.2777777777777778 0.375 rpy=0.0 0.0 0.0, axis 1 0 0, limit lower=0 upper=1.57 effort=5 velocity=2.283
- added joint handle8_to_drawer7: type fixed, parent drawer7, child handle8, origin xyz=0 0.16666666666666666 0.125 rpy=1.5707963267948963 0.0 0.0, axis 0 0 1, limit lower=0 upper=1.57 effort=5 velocity=2.283
- added joint handle9_to_drawer6: type fixed, parent drawer6, child handle9, origin xyz=0 0.16666666666666666 0.125 rpy=1.5707963267948963 0.0 0.0, axis 0 0 1, limit lower=0 upper=1.57 effort=5 velocity=2.283
- joint drawer2_to_base_link: origin xyz=0 0.3333333333333333 0.75 rpy=0.0 0.0 0.0 -> xyz=0 0.3333333333333333 0.0 rpy=0.0 0.0 0.0
- joint drawer3_to_base_link: origin xyz=0 0.3333333333333333 0.5 rpy=0.0 0.0 0.0 -> xyz=0 0.3333333333333333 0.25 rpy=0.0 0.0 0.0
- joint drawer4_to_base_link: origin xyz=0 0.3333333333333333 0.25 rpy=0.0 0.0 0.0 -> xyz=0 0.3333333333333333 0.5 rpy=0.0 0.0 0.0
- joint drawer5_to_base_link: origin xyz=0 0.3333333333333333 0.0 rpy=0.0 0.0 0.0 -> xyz=0 0.3333333333333333 0.75 rpy=0.0 0.0 0.0

File: output/label42.urdf (robot description, URDF)
Before this commit: robot my_urdf, 22 links, 21 joints
Links:
- removed link doorR2
- removed link drawer6
- added link doorR6, mass 0.2; collision mesh filename=../meshes/parts/doorR.obj scale=1 1.3233333333333333 1.6566666666666667; visual mesh filename=../meshes/parts/doorR.obj scale=1 1.3233333333333333 1.6566666666666667
- added link drawer2, mass 0.2; collision mesh filename=../meshes/parts/drawer.obj scale=1 0.6466666666666666 1.98; visual mesh filename=../meshes/parts/drawer.obj scale=1 0.6466666666666666 1.98
- link drawer0: geometry collision mesh filename=../meshes/parts/drawer.obj scale=1 2.3133333333333335 1.6466666666666667; visual mesh filename=../meshes/parts/drawer.obj scale=1 2.3133333333333335 1.6466666666666667
- link drawer1: geometry collision mesh filename=../meshes/parts/drawer.obj scale=1 1.3133333333333332 0.98; visual mesh filename=../meshes/parts/drawer.obj scale=1 1.3133333333333332 0.98
- link drawer3: geometry collision mesh filename=../meshes/parts/drawer.obj scale=1 0.6466666666666666 0.98; visual mesh filename=../meshes/parts/drawer.obj scale=1 0.6466666666666666 0.98
- link drawer4: geometry collision mesh filename=../meshes/parts/drawer.obj scale=1 0.98 0.98; visual mesh filename=../meshes/parts/drawer.obj scale=1 0.98 0.98
- link drawer5: geometry collision mesh filename=../meshes/parts/drawer.obj scale=1 1.3133333333333332 0.98; visual mesh filename=../meshes/parts/drawer.obj scale=1 1.3133333333333332 0.98
- link drawer7: geometry collision mesh filename=../meshes/parts/drawer.obj scale=1 1.98 0.98; visual mesh filename=../meshes/parts/drawer.obj scale=1 1.98 0.98
- link drawer8: geometry collision mesh filename=../meshes/parts/drawer.obj scale=1 1.6466666666666667 0.98; visual mesh filename=../meshes/parts/drawer.obj scale=1 1.6466666666666667 0.98
- link drawer9: geometry collision mesh filename=../meshes/parts/drawer.obj scale=1 1.98 0.98; visual mesh filename=../meshes/parts/drawer.obj scale=1 1.98 0.98
Joints:
- removed joint doorR2_to_base_link
- removed joint drawer14_to_drawer5
- removed joint drawer6_to_base_link
- removed joint knob11_to_drawer0
- removed joint knob12_to_drawer8
- removed joint knob13_to_drawer6
- removed joint knob15_to_drawer4
- removed joint knob16_to_drawer3
- removed joint knob17_to_doorR2
- removed joint knob18_to_drawer1
- removed joint knob19_to_drawer9
- added joint doorR6_to_base_link: type revolute, parent base_link, child doorR6, origin xyz=0 1.0 0.25 rpy=-0.0 -0.0 -0.0, axis 0 0 1, limit lower=0 upper=1.57 effort=5 velocity=2.283
- added joint drawer14_to_drawer3: type prismatic, parent drawer3, child drawer14, origin xyz=0 0.5 0.8333333333333334 rpy=0.0 0.0 0.0, axis 1 0 0, limit lower=0 upper=0.4 effort=5 velocity=2.283
- added joint drawer2_to_base_link: type prismatic, parent base_link, child drawer2, origin xyz=0 0.25 0.25 rpy=0.0 0.0 0.0, axis 1 0 0, limit lower=0 upper=0.4 effort=5 velocity=2.283
- added joint knob11_to_drawer4: type fixed, parent drawer4, child knob11, origin xyz=0 0.125 0.125 rpy=1.5707963267948963 0.0 0.0, axis 0 0 1, limit lower=0 upper=1.57 effort=5 velocity=2.283
- added joint knob12_to_drawer5: type fixed, parent drawer5, child knob12, origin xyz=0 0.16666666666666666 0.125 rpy=1.5707963267948963 0.0 0.0, axis 0 0 1, limit lower=0 upper=1.57 effort=5 velocity=2.283
- added joint knob13_to_drawer1: type fixed, parent drawer1, child knob13, origin xyz=0 0.16666666666666666 0.125 rpy=1.5707963267948963 0.0 0.0, axis 0 0 1, limit lower=0 upper=1.57 effort=5 velocity=2.283
- added joint knob15_to_drawer2: type fixed, parent drawer2, child knob15, origin xyz=0 0.08333333333333333 0.25 rpy=1.5707963267948963 0.0 0.0, axis 0 0 1, limit lower=0 upper=1.57 effort=5 velocity=2.283
- added joint knob16_to_drawer7: type fixed, parent drawer7, child knob16, origin xyz=0 0.25 0.125 rpy=1.5707963267948963 0.0 0.0, axis 0 0 1, limit lower=0 upper=1.57 effort=5 velocity=2.283
- added joint knob17_to_doorR6: type fixed, parent doorR6, child knob17, origin xyz=0 -0.2777777777777778 0.34722222222222227 rpy=0.0 0.0 0.0, axis 1 0 0, limit lower=0 upper=1.57 effort=5 velocity=2.283
- added joint knob18_to_drawer9: type fixed, parent drawer9, child knob18, origin xyz=0 0.25 0.125 rpy=1.5707963267948963 0.0 0.0, axis 0 0 1, limit lower=0 upper=1.57 effort=5 velocity=2.283
- added joint knob19_to_drawer8: type fixed, parent drawer8, child knob19, origin xyz=0 0.20833333333333334 0.125 rpy=1.5707963267948963 0.0 0.0, axis 0 0 1, limit lower=0 upper=1.57 effort=5 velocity=2.283
- joint drawer0_to_base_link: origin xyz=0 0.0 0.75 rpy=0.0 0.0 0.0 -> xyz=0 0.4166666666666667 0.25 rpy=0.0 0.0 0.0
- joint drawer1_to_base_link: origin xyz=0 0.5 0.0 rpy=0.0 0.0 0.0 -> xyz=0 0.0 0.25 rpy=0.0 0.0 0.0
- joint drawer3_to_base_link: origin xyz=0 0.0 0.0 rpy=0.0 0.0 0.0 -> xyz=0 0.0 0.5 rpy=0.0 0.0 0.0
- joint drawer4_to_base_link: origin xyz=0 0.25 0.25 rpy=0.0 0.0 0.0 -> xyz=0 0.0 0.75 rpy=0.0 0.0 0.0
- joint drawer5_to_base_link: origin xyz=0 0.0 0.5 rpy=0.0 0.0 0.0 -> xyz=0 0.3333333333333333 0.25 rpy=0.0 0.0 0.0
- joint drawer7_to_base_link: origin xyz=0 0.4166666666666667 0.25 rpy=0.0 0.0 0.0 -> xyz=0 0.0 0.0 rpy=0.0 0.0 0.0
- joint drawer8_to_base_link: origin xyz=0 0.3333333333333333 0.25 rpy=0.0 0.0 0.0 -> xyz=0 0.25 0.75 rpy=0.0 0.0 0.0
- joint drawer9_to_base_link: origin xyz=0 0.25 0.75 rpy=0.0 0.0 0.0 -> xyz=0 0.5 0.0 rpy=0.0 0.0 0.0
- joint knob20_to_drawer10: limit lower=0 upper=0.4 effort=5 velocity=2.283 -> lower=0 upper=1.57 effort=5 velocity=2.283

File: output/label53.urdf (robot description, URDF)
Before this commit: robot my_urdf, 11 links, 10 joints
Joints:
- removed joint handle5_to_drawer0
- removed joint handle6_to_drawer1
- removed joint handle7_to_drawer2
- added joint handle5_to_drawer2: type fixed, parent drawer2, child handle5, origin xyz=0 0.25 0.125 rpy=1.5707963267948963 0.0 0.0, axis 0 0 1, limit lower=0 upper=1.57 effort=5 velocity=2.283
- added joint handle6_to_drawer0: type fixed, parent drawer0, child handle6, origin xyz=0 0.25 0.125 rpy=1.5707963267948963 0.0 0.0, axis 0 0 1, limit lower=0 upper=1.57 effort=5 velocity=2.283
- added joint handle7_to_drawer1: type fixed, parent drawer1, child handle7, origin xyz=0 0.25 0.125 rpy=1.5707963267948963 0.0 0.0, axis 0 0 1, limit lower=0 upper=1.57 effort=5 velocity=2.283
- joint drawer0_to_base_link: origin xyz=0 0.5 0.75 rpy=0.0 0.0 0.0 -> xyz=0 0.5 0.5 rpy=0.0 0.0 0.0
- joint drawer1_to_base_link: origin xyz=0 0.5 0.5 rpy=0.0 0.0 0.0 -> xyz=0 0.5 0.25 rpy=0.0 0.0 0.0
- joint drawer2_to_base_link: origin xyz=0 0.5 0.25 rpy=0.0 0.0 0.0 -> xyz=0 0.5 0.75 rpy=0.0 0.0 0.0

File: output/label55.urdf (robot description, URDF)
Before this commit: robot my_urdf, 15 links, 14 joints
Links:
- removed link doorL5
- removed link doorR6
- removed link drawer2
- removed link drawer3
- added link doorL3, mass 0.2; collision mesh filename=../meshes/parts/doorL.obj scale=1 1.3233333333333333 2.6566666666666667; visual mesh filename=../meshes/parts/doorL.obj scale=1 1.3233333333333333 2.6566666666666667
- added link doorR2, mass 0.2; collision mesh filename=../meshes/parts/doorR.obj scale=1 1.3233333333333333 2.6566666666666667; visual mesh filename=../meshes/parts/doorR.obj scale=1 1.3233333333333333 2.6566666666666667
- added link drawer5, mass 0.2; collision mesh filename=../meshes/parts/drawer.obj scale=1 1.3133333333333332 0.98; visual mesh filename=../meshes/parts/drawer.obj scale=1 1.3133333333333332 0.98
- added link drawer6, mass 0.2; collision mesh filename=../meshes/parts/drawer.obj scale=1 1.3133333333333332 1.3133333333333332; visual mesh filename=../meshes/parts/drawer.obj scale=1 1.3133333333333332 1.3133333333333332
Joints:
- removed joint doorL5_to_base_link
- removed joint doorR6_to_base_link
- removed joint drawer2_to_base_link
- removed joint drawer3_to_base_link
- removed joint handle10_to_drawer3
- removed joint handle8_to_drawer1
- removed joint handle9_to_drawer2
- removed joint knob12_to_doorL5
- removed joint knob13_to_doorR6
- added joint doorL3_to_base_link: type revolute, parent base_link, child doorL3, origin xyz=0 0.3333333333333333 0.3333333333333333 rpy=0.0 0.0 0.0, axis 0 0 1, limit lower=-1.57 upper=0 effort=5 velocity=2.283
- added joint doorR2_to_base_link: type revolute, parent base_link, child doorR2, origin xyz=0 1.0 0.3333333333333333 rpy=-0.0 -0.0 -0.0, axis 0 0 1, limit lower=0 upper=1.57 effort=5 velocity=2.283
- added joint drawer5_to_base_link: type prismatic, parent base_link, child drawer5, origin xyz=0 0.0 0.25 rpy=0.0 0.0 0.0, axis 1 0 0, limit lower=0 upper=0.4 effort=5 velocity=2.283
- added joint drawer6_to_base_link: type prismatic, parent base_link, child drawer6, origin xyz=0 0.0 0.0 rpy=0.0 0.0 0.0, axis 1 0 0, limit lower=0 upper=0.4 effort=5 velocity=2.283
- added joint handle10_to_drawer1: type fixed, parent drawer1, child handle10, origin xyz=0 0.16666666666666666 0.125 rpy=1.5707963267948963 0.0 0.0, axis 0 0 1, limit lower=0 upper=1.57 effort=5 velocity=2.283
- added joint handle8_to_drawer5: type fixed, parent drawer5, child handle8, origin xyz=0 0.16666666666666666 0.125 rpy=1.5707963267948963 0.0 0.0, axis 0 0 1, limit lower=0 upper=1.57 effort=5 velocity=2.283
- added joint handle9_to_drawer6: type fixed, parent drawer6, child handle9, origin xyz=0 0.16666666666666666 0.16666666666666666 rpy=1.5707963267948963 0.0 0.0, axis 0 0 1, limit lower=0 upper=1.57 effort=5 velocity=2.283
- added joint knob12_to_doorL3: type fixed, parent doorL3, child knob12, origin xyz=0 0.2777777777777778 0.5555555555555556 rpy=0.0 0.0 0.0, axis 1 0 0, limit lower=0 upper=1.57 effort=5 velocity=2.283
- added joint knob13_to_doorR2: type fixed, parent doorR2, child knob13, origin xyz=0 -0.2777777777777778 0.5555555555555556 rpy=0.0 0.0 0.0, axis 1 0 0, limit lower=0 upper=1.57 effort=5 velocity=2.283
- joint drawer1_to_base_link: origin xyz=0 0.0 0.25 rpy=0.0 0.0 0.0 -> xyz=0 0.0 0.5 rpy=0.0 0.0 0.0
